File: IOT/практика/smart_watch/smart_watch.kicad_pcb (KiCad board)
At the start: 2 copper layers, 0 parts

Commit message: feat: adding hws and iot
Parts:
- added C1: 22uF, Capacitor_SMD:C_0603_1608Metric, F.Cu at (99.5, 91.5)
- added C2: 10nF, Capacitor_SMD:C_0603_1608Metric, F.Cu at (99.4, 97.4)
- added C3: 22uF, Capacitor_SMD:C_0603_1608Metric, F.Cu at (99.4, 99.9)
- added C4: 22uF, Capacitor_SMD:C_0603_1608Metric, F.Cu at (99.4, 102.4)
- added C5: 22uF, Capacitor_SMD:C_0603_1608Metric, F.Cu at (99.4, 105.0)
- added C6: 1uF, Capacitor_SMD:C_0603_1608Metric, F.Cu at (99.4, 107.5)
- added C7: 1uF, Capacitor_SMD:C_0603_1608Metric, F.Cu at (103.5, 91.5)
- added C8: 100nF, Capacitor_SMD:C_0603_1608Metric, F.Cu at (103.5, 97.4)
- added D1: LED, LED_SMD:LED_0603_1608Metric, F.Cu at (117.0, 111.0)
- added D2: LED, LED_SMD:LED_0603_1608Metric, F.Cu at (117.0, 102.0)
- added J1: Conn_01x02_Pin, TerminalBlock:TerminalBlock_MaiXu_MX126-5.0-02P_1x02_P5.00mm, F.Cu at (125.2, 99.5)
- added J2: USB_C_Receptacle_USB2.0_16P, Connector_USB:USB_C_Receptacle_Amphenol_124019772112A, F.Cu at (117.0, 133.0)
- added L1: 1.0uH, Inductor_SMD:L_Changjiang_FXL0630, F.Cu at (151.5, 110.5)
- added R1: 203k, Resistor_SMD:R_0603_1608Metric, F.Cu at (103.5, 99.9)
- added R10: 10k, Resistor_SMD:R_0603_1608Metric, F.Cu at (107.5, 105.0)
- added R2: 100k, Resistor_SMD:R_0603_1608Metric, F.Cu at (103.5, 102.4)
- added R3: 1.0Meg, Resistor_SMD:R_0603_1608Metric, F.Cu at (103.5, 105.0)
- added R4: 1k, Resistor_SMD:R_0603_1608Metric, F.Cu at (103.5, 107.5)
- added R5: 2k, Resistor_SMD:R_0603_1608Metric, F.Cu at (107.5, 91.5)
- added R6: 1.5k, Resistor_SMD:R_0603_1608Metric, F.Cu at (107.5, 97.4)
- added R7: 10k, Resistor_SMD:R_0603_1608Metric, F.Cu at (107.5, 99.9)
- added R8: 1.5k, Resistor_SMD:R_0603_1608Metric, F.Cu at (107.5, 102.4)
- added SW3: SW_Push, Button_Switch_SMD:SW_Push_1P1T_NO_CK_KMR2, F.Cu at (143.0, 90.0)
- added U3: KXTJ3-1057, Package_LGA:Kionix_LGA-12_2x2mm_P0.5mm_LayoutBorder2x4y, F.Cu at (158.2, 98.8)
- added U4: MAX30102, OptoDevice:Maxim_OLGA-14_3.3x5.6mm_P0.8mm, F.Cu at (136.6, 97.3)
- added U5: TPS61230DRC, Package_SON:Texas_S-PVSON-N10_ThermalVias, F.Cu at (139.8, 123.0)
- added U6: BQ24090DGQ, Package_SO:HVSSOP-10-1EP_3x3mm_P0.5mm_EP1.57x1.88mm_ThermalVias, F.Cu at (111.0, 116.5)
- added U7: ESP32-WROOM-32, RF_Module:ESP32-WROOM-32, F.Cu at (122.0, 82.6)
