File: IOT/практика/smart_watch/smart_watch.kicad_pcb (KiCad board)
At the start: 2 copper layers, 28 parts, among them J1 Conn_01x02_Pin, J2 USB_C_Receptacle_USB2.0_16P, SW3 SW_Push, U3 KXTJ3-1057, U4 MAX30102, U5 TPS61230DRC, U6 BQ24090DGQ, U7 ESP32-WROOM-32

Commit message: feat: adding things
Parts:
- added U1: ~, Connector_FFC:Hirose_FH12-13S-0.5SH_1x13-1MP_P0.50mm_Horizontal, F.Cu at (104.0, 105.5)
- moved U3 62.4 mm to (97.8, 114.2)
- moved SW3 61.9 mm to (101.0, 135.5)
- moved C1 57.1 mm to (147.0, 123.3), turned to -90 degrees
- moved C2 56.8 mm to (150.0, 123.3), turned to -90 degrees
- moved J1 36.5 mm to (137.0, 134.0)
- moved R3 35.9 mm to (133.2, 125.0)
- moved R2 34.8 mm to (133.2, 120.5)
- moved R1 34.6 mm to (129.2, 123.0)
- moved R5 28.7 mm to (117.2, 118.5)
- moved C7 28.2 mm to (113.2, 118.0)
- moved R10 25.8 mm to (103.8, 130.5)
- moved R6 25.1 mm to (121.2, 118.5)
- moved D2 23.2 mm to (125.7, 123.5)
- moved C3 22.2 mm to (102.2, 122.0)
- moved C4 22.1 mm to (109.7, 122.0)
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Connections:
- U7 pad 13: unconnected-(U7-IO14-Pad13) -> LCD_BL
- U7 pad 14: unconnected-(U7-IO12-Pad14) -> LCD_DC
- U7 pad 16: unconnected-(U7-IO13-Pad16) -> LCD_RST
- U7 pad 23: unconnected-(U7-IO15-Pad23) -> TP_INT
- U7 pad 27: unconnected-(U7-IO16-Pad27) -> TP_RST
- U7 pad 29: CS -> LCD_CS
- U7 pad 31: unconnected-(U7-IO19-Pad31) -> MISO
Routing:
- net GNDD: track 0.00 -> 16.5 mm

Commit message: updating smart watch
Parts:
- added C10: 0.1 uF, Capacitor_SMD:C_0603_1608Metric, F.Cu at (142.5, 107.0)
- added C16: 1uF, Capacitor_SMD:C_0603_1608Metric, F.Cu at (140.7, 95.0)
- added C9: 0.1 uF, Capacitor_SMD:C_0603_1608Metric, F.Cu at (139.5, 107.0)
- added R11: 10K, Resistor_SMD:R_0603_1608Metric, F.Cu at (133.0, 107.0)
- added R12: 10K, Resistor_SMD:R_0603_1608Metric, F.Cu at (135.0, 96.0)
- added R13: 10K, Resistor_SMD:R_0603_1608Metric, F.Cu at (132.0, 91.5)
- added R14: 10K, Resistor_SMD:R_0603_1608Metric, F.Cu at (132.0, 94.5)
- added R15: 10K, Resistor_SMD:R_0603_1608Metric, F.Cu at (103.0, 94.0)
- added R16: 10K, Resistor_SMD:R_0603_1608Metric, F.Cu at (105.0, 94.0)
- added R9: 10K, Resistor_SMD:R_0603_1608Metric, F.Cu at (138.0, 96.5)
- added SW4: SW_Push, Button_Switch_SMD:SW_Push_1P1T_NO_CK_KMR2, F.Cu at (111.0, 125.5)
- added U10: NLSV2T244D, Package_SO:SOIC-8_3.9x4.9mm_P1.27mm, F.Cu at (134.5, 101.0)
- added U2: CH330N, Package_SO:SOIC-8_3.9x4.9mm_P1.27mm, F.Cu at (135.0, 112.0)
- added U8: LC709203FQH-01TWG, Package_DFN_QFN:WDFN-8-1EP_4x3mm_P0.65mm_EP2.4x1.8mm, F.Cu at (137.6, 91.5)
- moved SW3 42.7 mm to (139.5, 117.0)
- moved R10 40.3 mm to (109.0, 90.5)
- moved C1 33.1 mm to (115.5, 113.0), turned to 90 degrees
- moved C2 28.9 mm to (123.0, 113.0), turned to 90 degrees
- moved C3 25.0 mm to (125.5, 113.0), turned to 90 degrees
- moved U5 24.8 mm to (119.0, 113.0)
- moved U3 23.0 mm to (108.2, 93.8)
- moved D2 22.3 mm to (106.5, 112.2), turned to 180 degrees
- moved R8 22.0 mm to (103.5, 113.0), turned to -90 degrees
- moved R6 20.4 mm to (101.5, 113.0), turned to -90 degrees
- moved L1 19.7 mm to (119.5, 119.0)
- moved D1 19.1 mm to (99.5, 112.8), turned to 90 degrees
- moved C8 16.0 mm to (98.5, 108.5)
- moved J1 15.1 mm to (128.5, 121.5)
- moved U6 14.3 mm to (107.1, 117.0)
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Connections:
- net Net-(U6-IN) renamed VBUS
- J2 pad A6: unconnected-(J2-D+-PadA6) -> D+
- J2 pad A7: unconnected-(J2-D--PadA7) -> D-
- R10 pad 1: Net-(U7-EN) -> +3V3
- R10 pad 2: GNDD -> Net-(U7-EN)
- SW3 pad 1: +3V3 -> GNDD
- U4 pad 11: 3V3 -> +3V3
- U7 pad 25: unconnected-(U7-IO0-Pad25) -> BOOT
- U7 pad 26: unconnected-(U7-IO4-Pad26) -> TP_RST
- U7 pad 27: TP_RST -> RX_2
- U7 pad 28: unconnected-(U7-IO17-Pad28) -> TX_2
- U7 pad 35: unconnected-(U7-TXD0/IO1-Pad35) -> TX
Routing:
- net GNDD: track 16.5 -> 0.00 mm
Other:
- board outline added: 49.6 x 49.6 mm
- board text added: "Designed by Bobi and Yo"

Commit message: updating smart watch
Parts:
- moved R10 1.66 mm to (107.3, 90.5), turned to 180 degrees
- moved R15 1.66 mm to (101.3, 94.0)
- moved R16 1.66 mm to (103.3, 94.0)
- moved U3 1.66 mm to (106.6, 93.8)
- moved C4 1.50 mm to (105.0, 120.0)
- moved C1 1.12 mm to (114.5, 113.5)
- moved C6 0.71 mm to (113.5, 119.3)
- moved R4 0.71 mm to (112.0, 119.0)
- moved U8 0.70 mm to (136.9, 91.5)
- moved C2 0.50 mm to (123.5, 113.0)
- moved C5 0.50 mm to (101.5, 117.8)
- moved SW3 0.50 mm to (139.5, 116.5)
- moved C16 0.28 mm to (141.0, 95.0)
Connections:
- U7 pad 27: RX_2 -> unconnected-(U7-IO16-Pad27)
- U7 pad 28: TX_2 -> unconnected-(U7-IO17-Pad28)
Routing:
- net GNDD: track 0.00 -> 250.3 mm, vias 0 -> 16
- net V_BAIT: track 0.00 -> 108.9 mm, vias 0 -> 13
- net SCL: track 0.00 -> 92.2 mm, vias 0 -> 5
- net 3.3V_OUT: track 0.00 -> 84.4 mm, vias 0 -> 8
- net VBUS: track 0.00 -> 73.6 mm, vias 0 -> 6
- net SDA: track 0.00 -> 65.0 mm, vias 0 -> 5
- net Net-(U7-EN): track 0.00 -> 61.8 mm, vias 0 -> 4
- net +3V3: track 0.00 -> 56.8 mm, vias 0 -> 4
- net MOSI: track 0.00 -> 40.7 mm, vias 0 -> 4
- net TP_INT: track 0.00 -> 38.6 mm, vias 0 -> 4
- net BOOT: track 0.00 -> 38.1 mm, vias 0 -> 2
- net TP_RST: track 0.00 -> 33.0 mm, vias 0 -> 4
- net MISO: track 0.00 -> 30.6 mm, vias 0 -> 2
- net SCK: track 0.00 -> 28.8 mm, vias 0 -> 2
- net LCD_CS: track 0.00 -> 27.6 mm, vias 0 -> 2
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